Commit message: update ui2024 - NOTICE: might fix a prev tf issue

File: bluerov_model/BlueRov2_TBNMS.urdf.xacro (robot description, xacro)
@@ -82,5 +82,5 @@
       <origin xyz="0 0 0.07" rpy="-3.141592653589793 3.141592653589793 1.5707963267948966" />
       <geometry>
-        <mesh filename="package://bluerov_state_estimation/bluerov_model/BlueRov2.dae" />
+        <mesh filename="package://bluerov_visualizer/bluerov_model/BlueRov2.dae" />
       </geometry>
     </visual>
@@ -225,4 +225,5 @@
     <origin rpy="0 0 0" xyz="0.0 0.03 0" />
   </joint>
+<!-- TODO: Jingyu - this transformation might be wrong!!! -->
   <!-- ZEDM Left Camera Optical Frame -->
   <link name="zedm_left_camera_optical_frame" />

File: bluerov_model/BlueRov2_UI2024.urdf.xacro (robot description, xacro)
@@ -174,5 +174,4 @@
     <origin rpy="0 0 0" xyz="0 0 0" />
   </joint>
-  <!-- DVL -->
   <link name="dvl_link"></link>
   <joint name="dvl_joint" type="fixed">
@@ -181,5 +180,4 @@
     <origin rpy="0 0 0.0505" xyz="0.16443882752 0.00429 0.28362510322" />
   </joint>
-  <!-- Transducer 1 -->
   <link name="transducer1_link"></link>
   <joint name="transducer1_joint" type="fixed">
@@ -188,5 +186,4 @@
     <origin rpy="-0.28492413 -0.2740142 0.0395455" xyz="-0.01385929 0.01385929 -0.00555" />
   </joint>
-  <!-- Transducer 2 -->
   <link name="transducer2_link"></link>
   <joint name="transducer2_joint" type="fixed">
@@ -195,5 +192,4 @@
     <origin rpy="0.28492413 -0.2740142 -0.0395455" xyz="-0.01385929 -0.01385929 -0.00555" />
   </joint>
-  <!-- Transducer 3 -->
   <link name="transducer3_link"></link>
   <joint name="transducer3_joint" type="fixed">
@@ -202,5 +198,4 @@
     <origin rpy="0.28492413 0.2740142 0.0395455" xyz="0.01385929 -0.01385929 -0.00555" />
   </joint>
-  <!-- Transducer 4 -->
   <link name="transducer4_link"></link>
   <joint name="transducer4_joint" type="fixed">
@@ -214,5 +209,5 @@
     <parent link="base_link" />
     <child link="zedm_base_link" />
-    <origin rpy="0.0318 -1.5708 0.0" xyz="-0.1234754910177292 -0.12034209908167565 0.28534500108" />
+    <origin rpy="0.0 -1.5707963267948966 1.5707963267948966" xyz="0.00252551 -0.06238885 0.26832" />
   </joint>
   <!-- ZEDM Camera Center -->
@@ -230,4 +225,5 @@
     <origin rpy="0 0 0" xyz="0.0 0.03 0" />
   </joint>
+<!-- Jingyu: fix a possiblely wrong tf - might lead to wrong tf from the  -->
   <!-- ZEDM Left Camera Optical Frame -->
   <link name="zedm_left_camera_optical_frame" />
@@ -235,5 +231,5 @@
     <parent link="zedm_left_camera_frame" />
     <child link="zedm_left_camera_optical_frame" />
-    <origin rpy="-1.5707963 1.5707963 0" xyz="0 0 0" />
+    <origin rpy="-1.5707963 0 -1.5707963" xyz="0 0 0" />
   </joint>
   <!-- ZEDM Right Camera Frame -->
@@ -244,4 +240,5 @@
     <origin rpy="0 0 0" xyz="0.0 -0.03 0" />
   </joint>
+<!-- Jingyu: fix a possiblely wrong tf - might lead to wrong tf from the  -->
   <!-- ZEDM Right Camera Optical Frame -->
   <link name="zedm_right_camera_optical_frame" />
@@ -249,5 +246,5 @@
     <parent link="zedm_right_camera_frame" />
     <child link="zedm_right_camera_optical_frame" />
-    <origin rpy="-1.5707963 1.5707963 0" xyz="0 0 0" />
+    <origin rpy="-1.5707963 0 -1.5707963" xyz="0 0 0" />
   </joint>
   <!-- ZEDM IMU Link -->
@@ -259,4 +256,29 @@
       xyz="-0.0020000000949949026 -0.015000001527369022 -0.0017100002150982618" />
   </joint>
+  <!-- VISUALIZATION PURPOSES -->
+  <link name="transducer1_link_viz"></link>
+  <joint name="transducer1_joint_viz" type="fixed">
+    <parent link="dvl_link" />
+    <child link="transducer1_link_viz" />
+    <origin rpy="-2.3562   -1.1781    2.3562" xyz="-0.01385929 0.01385929 -0.00555" />
+  </joint>
+  <link name="transducer2_link_viz"></link>
+  <joint name="transducer2_joint_viz" type="fixed">
+    <parent link="dvl_link" />
+    <child link="transducer2_link_viz" />
+    <origin rpy="2.3562   -1.1781   -2.3562" xyz="-0.01385929 -0.01385929 -0.00555" />
+  </joint>
+  <link name="transducer3_link_viz"></link>
+  <joint name="transducer3_joint_viz" type="fixed">
+    <parent link="dvl_link" />
+    <child link="transducer3_link_viz" />
+    <origin rpy="0.7854 -1.1781 -0.7854" xyz="0.01385929 -0.01385929 -0.00555" />
+  </joint>
+  <link name="transducer4_link_viz"></link>
+  <joint name="transducer4_joint_viz" type="fixed">
+    <parent link="dvl_link" />
+    <child link="transducer4_link_viz" />
+    <origin rpy="-0.7854   -1.1781    0.7854" xyz="0.01385929 0.01385929 -0.00555" />
+  </joint>
   <!-- Sonar -->
   <link name="sonar_link"></link>
@@ -264,5 +286,5 @@
     <parent link="base_link" />
     <child link="sonar_link" />
-    <origin rpy="0 0 0" xyz="-0.14902354966 0.0936 0.30638500108" />
+    <origin rpy="0 0 0" xyz="0.164107 0.10618 0.30638500108" />
   </joint>
   <link name="sonar_link_viz"></link>
@@ -270,30 +292,5 @@
     <parent link="base_link" />
     <child link="sonar_link_viz" />
-    <origin rpy="3.1416 -1.5708 0.0" xyz="-0.14902354966 0.0936 0.30638500108" />
-  </joint>
-  <!-- VISUALIZATION PURPOSES -->
-  <link name="transducer1_link_viz"></link>
-  <joint name="transducer1_joint_viz" type="fixed">
-    <parent link="dvl_link" />
-    <child link="transducer1_link_viz" />
-    <origin rpy="-2.3562   -1.1781    2.3562" xyz="-0.01385929 0.01385929 -0.00555" />
-  </joint>
-  <link name="transducer2_link_viz"></link>
-  <joint name="transducer2_joint_viz" type="fixed">
-    <parent link="dvl_link" />
-    <child link="transducer2_link_viz" />
-    <origin rpy="2.3562   -1.1781   -2.3562" xyz="-0.01385929 -0.01385929 -0.00555" />
-  </joint>
-  <link name="transducer3_link_viz"></link>
-  <joint name="transducer3_joint_viz" type="fixed">
-    <parent link="dvl_link" />
-    <child link="transducer3_link_viz" />
-    <origin rpy="0.7854 -1.1781 -0.7854" xyz="0.01385929 -0.01385929 -0.00555" />
-  </joint>
-  <link name="transducer4_link_viz"></link>
-  <joint name="transducer4_joint_viz" type="fixed">
-    <parent link="dvl_link" />
-    <child link="transducer4_link_viz" />
-    <origin rpy="-0.7854   -1.1781    0.7854" xyz="0.01385929 0.01385929 -0.00555" />
+    <origin rpy="3.1416   -1.5708         0" xyz="0.164107 0.10618 0.30638500108" />
   </joint>
 </robot>
