Commit message: udpate latest config

File: bluerov_model/BlueRov2_UI2024.urdf.xacro (robot description, xacro)
@@ -211,4 +211,10 @@
     <origin rpy="0.0 -1.5707963267948966 1.5707963267948966" xyz="0.00252551 -0.06238885 0.26832" />
   </joint>
+  <!-- <link name="zedm_base_link" />
+  <joint name="zedm_base_joint" type="fixed">
+    <parent link="base_link" />
+    <child link="zedm_base_link" />
+    <origin rpy="-1.5707963267948966 0.0 1.5707963267948966" xyz="0.00252551 -0.06238885 0.26832" />
+  </joint> -->
   <!-- ZEDM Camera Center -->
   <link name="zedm_camera_center" />
@@ -256,4 +262,18 @@
       xyz="-0.0020000000949949026 -0.015000001527369022 -0.0017100002150982618" />
   </joint>
+ <link name="sensor" />
+  <joint name="sensor_joint" type="fixed">
+    <parent link="zedm_left_camera_optical_frame" />
+    <child link="sensor" />
+    <origin rpy="-1.5577479 0.0030325 -1.5733366"
+      xyz="0.07989305 0.08146287 -0.02610534" />
+  </joint>
+  <link name="sensor_wgs84" />
+  <joint name="sensor_wgs84_joint" type="fixed">
+    <parent link="zedm_left_camera_optical_frame" />
+    <child link="sensor_wgs84" />
+    <origin rpy="-1.5577479 0.0030325 -1.5733366"
+      xyz="0.07989305 0.08146287 -0.02610534" />
+  </joint>
   <!-- VISUALIZATION PURPOSES -->
   <link name="transducer1_link_viz"></link>
